Commit message: update tcp in urdf to max optimal umi setup

File: urdf/panda/panda.urdf (robot description, URDF)
Before this commit: robot panda, 22 links, 21 joints
Joints:
- joint panda_hand_tcp_joint: origin xyz=0 0 0.1034 rpy=0 0 0 -> xyz=0 0 0.1934 rpy=0 0 0

Commit message: reverse tcp for testing

File: urdf/panda/panda.urdf (robot description, URDF)
Before this commit: robot panda, 22 links, 21 joints
Joints:
- joint panda_hand_tcp_joint: origin xyz=0 0 0.1934 rpy=0 0 0 -> xyz=0 0 0.1034 rpy=0 0 0
